Commit message: can rotate angle

File: excurate_arm/target.urdf (robot description, URDF)
Before this commit: robot angle_excurate_arm_ver2, 7 links, 6 joints
Links:
- link base_link: geometry collision mesh filename=package://angle_excurate_arm_ver2_description/meshes/base_l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 scale=0.001 0.001 0.001; visual mesh filename=package://angle_excurate_arm_ver2_description/meshes/base_l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 scale=0.001 0.001 0.001
- link base_link2_v2_1: geometry collision mesh filename=package://angle_excurate_arm_ver2_description/meshes/base_l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 scale=0.001 0.001 0.001; visual mesh filename=package://angle_excurate_arm_ver2_description/meshes/base_l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 scale=0.001 0.001 0.001
- link link3_v1_1: geometry collision mesh filename=package://angle_excurate_arm_ver2_description/meshes/link3_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 scale=0.001 0.001 0.001; visual mesh filename=package://angle_excurate_arm_ver2_description/meshes/link3_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 scale=0.001 0.001 0.001
- link link4_v1_1: geometry collision mesh filename=package://angle_excurate_arm_ver2_description/meshes/link4_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 scale=0.001 0.001 0.001; visual mesh filename=package://angle_excurate_arm_ver2_description/meshes/link4_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 scale=0.001 0.001 0.001
- link robot_ver7_grap1_2_v1_1: geometry collision mesh filename=package://angle_excurate_arm_ver2_description/meshes/robot_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 scale=0.001 0.001 0.001; visual mesh filename=package://angle_excurate_arm_ver2_description/meshes/robot_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 scale=0.001 0.001 0.001
- link robot_ver7_grap2_2_v1_1: geometry collision mesh filename=package://angle_excurate_arm_ver2_description/meshes/robot_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 scale=0.001 0.001 0.001; visual mesh filename=package://angle_excurate_arm_ver2_description/meshes/robot_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 scale=0.001 0.001 0.001
- link robot_ver7_link_4_v1_1: geometry collision mesh filename=package://angle_excurate_arm_ver2_description/meshes/robot_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 scale=0.001 0.001 0.001; visual mesh filename=package://angle_excurate_arm_ver2_description/meshes/robot_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 scale=0.001 0.001 0.001

Commit message: add drake

File: excurate_arm/target.urdf (robot description, URDF)
Before this commit: robot angle_excurate_arm_ver2, 7 links, 6 joints
Links:
- link base_link: geometry collision mesh filename=meshes/base_link.obj scale=0.001 0.001 0.001; visual mesh filename=meshes/base_link.obj scale=0.001 0.001 0.001
- link base_link2_v2_1: geometry collision mesh filename=meshes/base_link2_v2_1.obj scale=0.001 0.001 0.001; visual mesh filename=meshes/base_link2_v2_1.obj scale=0.001 0.001 0.001
- link link3_v1_1: geometry collision mesh filename=meshes/link3_v1_1.obj scale=0.001 0.001 0.001; visual mesh filename=meshes/link3_v1_1.obj scale=0.001 0.001 0.001
- link link4_v1_1: geometry collision mesh filename=meshes/link4_v1_1.obj scale=0.001 0.001 0.001; visual mesh filename=meshes/link4_v1_1.obj scale=0.001 0.001 0.001
- link robot_ver7_grap1_2_v1_1: geometry collision mesh filename=meshes/robot_ver7_grap1_2_v1_1.obj scale=0.001 0.001 0.001; visual mesh filename=meshes/robot_ver7_grap1_2_v1_1.obj scale=0.001 0.001 0.001
- link robot_ver7_grap2_2_v1_1: geometry collision mesh filename=meshes/robot_ver7_grap2_2_v1_1.obj scale=0.001 0.001 0.001; visual mesh filename=meshes/robot_ver7_grap2_2_v1_1.obj scale=0.001 0.001 0.001
- link robot_ver7_link_4_v1_1: geometry collision mesh filename=meshes/robot_ver7_link_4_v1_1.obj scale=0.001 0.001 0.001; visual mesh filename=meshes/robot_ver7_link_4_v1_1.obj scale=0.001 0.001 0.001
Joints:
- joint Revolute 6: mimic joint=Revolute 5 multiplier=-1.0 -> (none)

Commit message: change urdf base link to world

File: excurate_arm/target.urdf (robot description, URDF)
Before this commit: robot angle_excurate_arm_ver2, 7 links, 6 joints
Links:
- added link world
Joints:
- added joint floating_base: type floating, parent world, child base_link

Commit message: 實驗用 urdf

File: excurate_arm/target.urdf (robot description, URDF)
Before this commit: robot angle_excurate_arm_ver2, 8 links, 7 joints
Joints:
- removed joint floating_base
- added joint world_to_base: type fixed, parent world, child base_link, origin xyz=0 0 0 rpy=0 0 0

Commit message: change urdf both
new_config2's demo can use but other cannot

File: excurate_arm/target.urdf (robot description, URDF)
Before this commit: robot angle_excurate_arm_ver2, 8 links, 7 joints
Links:
- link world: geometry visual box size=0.1 0.1 0.1

File: moveit_docker_activate/src/robot_description/urdf/target.urdf (robot description, URDF)
Before this commit: robot angle_excurate_arm_ver2, 8 links, 7 joints
Joints:
- joint Revolute 1: origin xyz=2.989375 1.116433 0.075907 rpy=0 0 0 -> xyz=0.0 0.0 0.075907 rpy=0 0 0
