Commit message: add origin arm

File: moveit_docker_activate/install/robot_description/share/robot_description/urdf/target.urdf (robot description, URDF)
Before this commit: robot angle_excurate_arm_ver2, 7 links, 6 joints
Joints:
- joint Revolute 1: origin xyz=2.989375 1.116433 0.075907 rpy=0 0 0 -> xyz=0.0 0.0 0.075907 rpy=0 0 0

File: moveit_docker_activate/src/robot_description/urdf/target.urdf (robot description, URDF)
Before this commit: robot angle_excurate_arm_ver2, 8 links, 7 joints
Links:
- removed link world
Joints:
- removed joint world_joint
