Commit message: let moveit can use

File: moveit_docker_activate/src/robot_description_version2/urdf/target.urdf (robot description, URDF)
Before this commit: robot angle_excurate_arm_ver2, 8 links, 7 joints
Links:
- added link base_link_dummy, mass 1.0
- link base_link: mass 7.925585093654501e-07 -> None
Joints:
- added joint base_link_to_dummy: type fixed, parent base_link, child base_link_dummy, origin xyz=0 0 0 rpy=0 0 0
